Commit message: Change masses exercise 1

File: exercice1/double_pendulum.urdf (robot description, URDF)
Before this commit: robot pendulum, 5 links, 4 joints
Links:
- link PendulumMass: mass 3.0 -> 300.0
- link SecondPendulumMass: mass 2.0 -> 200.0

Commit message: Change torque and velocity limits

File: exercice1/double_pendulum.urdf (robot description, URDF)
Before this commit: robot pendulum, 5 links, 4 joints
Joints:
- joint PendulumJoint: limit lower=-100 upper=100 effort=1000 velocity=100 -> lower=-100 upper=100 effort=100000 velocity=10000
- joint SecondPendulumJoint: limit lower=-100 upper=100 effort=1000 velocity=100 -> lower=-100 upper=100 effort=100000 velocity=10000
